File: mini-bship.kicad_pcb (KiCad board)
At the start: 2 copper layers, 0 parts

Commit message: Slow progress, got started on pcb
Parts:
- added C1: 22pF, Capacitor_SMD:C_0805_2012Metric, F.Cu at (146.8, 64.8)
- added C2: 22pF, Capacitor_SMD:C_0805_2012Metric, F.Cu at (141.1, 68.1)
- added C3: 1uF, Capacitor_SMD:C_0805_2012Metric, F.Cu at (121.7, 88.5)
- added C4: 0.1uF, Capacitor_SMD:C_0805_2012Metric, F.Cu at (136.1, 75.1)
- added C5: 0.1uF, Capacitor_SMD:C_0805_2012Metric, F.Cu at (121.7, 85.6)
- added C6: 0.1uF, Capacitor_SMD:C_0805_2012Metric, F.Cu at (125.5, 82.6)
- added C7: 0.1uF, Capacitor_SMD:C_0805_2012Metric, F.Cu at (131.2, 78.4)
- added D1: D_Small, Diode_SMD:D_SOD-123, F.Cu at (47.0, 29.0)
- added D2: D_Small, Diode_SMD:D_SOD-123, F.Cu at (66.0, 29.0)
- added D3: D_Small, Diode_SMD:D_SOD-123, F.Cu at (47.0, 48.0)
- added D4: D_Small, Diode_SMD:D_SOD-123, F.Cu at (66.0, 48.0)
- added F1: 500mA, Fuse:Fuse_1206_3216Metric, F.Cu at (116.5, 89.1)
- added MX1: MX-NoLED, keyboard_parts:ALPS_PLATE_SPRING, F.Cu at (39.4, 29.3)
- added MX2: MX-NoLED, keyboard_parts:ALPS_PLATE_SPRING, F.Cu at (58.5, 29.3)
- added MX3: MX-NoLED, keyboard_parts:ALPS_PLATE_SPRING, F.Cu at (39.4, 48.4)
- added MX4: MX-NoLED, keyboard_parts:ALPS_PLATE_SPRING, F.Cu at (58.5, 48.4)
- added R1: 10k, Resistor_SMD:R_0805_2012Metric, F.Cu at (115.9, 96.7)
- added R2: 22, Resistor_SMD:R_0805_2012Metric, F.Cu at (141.1, 71.1)
- added R3: 22, Resistor_SMD:R_0805_2012Metric, F.Cu at (129.9, 82.6)
- added R4: 10k, Resistor_SMD:R_0805_2012Metric, F.Cu at (126.1, 85.5)
- added SW1: SW_Push, random-keyboard-parts:SKQG-1155865, F.Cu at (118.5, 80.9)
- added U1: ATmega32U4-AU, Package_QFP:TQFP-44_10x10mm_P0.8mm, F.Cu at (121.0, 70.5)
- added USB1: Molex-0548190589, random-keyboard-parts:Molex-0548190589, F.Cu at (132.5, 68.4)
- added Y1: 16MHz, Crystal:Crystal_SMD_3225-4Pin_3.2x2.5mm, F.Cu at (116.4, 93.0)
