File: mini-bship.sch (KiCad schematic (older format))
At the start: 16 parts

Commit message: Slow progress, got started on pcb
Parts:
- added D1, D2, D3, D4, D? (x6): D_Small, Diode_SMD:D_SOD-123, symbol Device:D_Small
- added K1, K2, K3, K4, K? (x6): MX-NoLED, keyboard_parts:ALPS_PLATE_SPRING, symbol MX_Alps_Hybrid:MX-NoLED
- C1, C2, C3, C4, C5, C6, C7: renamed from C?; footprint (none) -> Capacitor_SMD:C_0805_2012Metric
- F1: renamed from F?; footprint (none) -> Fuse:Fuse_1206_3216Metric
- R1, R2, R3, R4: renamed from R?; footprint (none) -> Resistor_SMD:R_0805_2012Metric
- SW1: renamed from SW?; footprint (none) -> random-keyboard-parts:SKQG-1155865
- USB1: renamed from USB?; footprint (none) -> random-keyboard-parts:Molex-0548190589
- Y1: renamed from Y?; footprint (none) -> Crystal:Crystal_SMD_3225-4Pin_3.2x2.5mm
- gave numbers to parts that had none: 1
Connections:
- new net: D1.2 (A), K1.2 (ROW)
- new net: D2.2 (A), K2.2 (ROW)
- new net: D3.2 (A), K3.2 (ROW)
- new net: D4.2 (A), K4.2 (ROW)
- new net: D?.2 (A), K?.2 (ROW) (x6)
- new net COL0: K1.1 (COL), K3.1 (COL), K?.1 (COL), K?.1 (COL), K?.1 (COL)
- new net COL1: K2.1 (COL), K4.1 (COL), K?.1 (COL), K?.1 (COL), K?.1 (COL)
- new net ROW0: D1.1 (K), D2.1 (K)
- new net ROW1: D3.1 (K), D4.1 (K)
- new net ROW2: D?.1 (K), D?.1 (K)
- new net ROW3: D?.1 (K), D?.1 (K)
- new net ROW4: D?.1 (K), D?.1 (K)
Other:
- moved on the sheet: C1, C2, C3, C4, C5, C6, C7, R1, R2, R3, R4, SW1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
